File: hardware/kicad/parts_servo3.kicad_pcb (KiCad board)
At the start: 2 copper layers, 37.3 x 17.5 mm, 49 parts, among them Q110 NFET-DUAL, Q120 NFET-DUAL, U1 MCP1703-3302, U100 RT9625A, U200 AS5050, U50 NRF51822, X60 16MHz

Commit message: Update PCB
Parts:
- added REF0011: Via, parts_servo:Via, F.Cu at (153.4, 97.9)
- added REF0012: Via, parts_servo:Via, F.Cu at (145.4, 99.2)
- added REF0013: Via, parts_servo:Via, F.Cu at (145.7, 107.3)
- added REF0014: Via, parts_servo:Via, F.Cu at (143.4, 107.3)
- added REF0015: Via, parts_servo:Via, F.Cu at (143.4, 105.2)
- added REF0016: Via, parts_servo:Via, F.Cu at (145.7, 105.2)
- moved L70 0.13 mm to (144.9, 102.0)
Routing:
- net Net-(L70-Pad1): track 2.28 -> 2.99 mm
- net GND: vias 9 -> 7
Other:
- rule pad_to_mask_clearance: 0 -> 0.0762
